File: stm32h753_dev.kicad_pcb (KiCad board)
At the start: 4 copper layers, 99.1 x 53.3 mm, 90 parts, among them J1 Conn_02x38_Counter_Clockwise, J2 Conn_02x38_Counter_Clockwise, J3 USB_C_Receptacle_USB2.0_16P, J4 USB_C_Receptacle_USB2.0_16P, J5 DE9_Pins_MountingHoles, J6 Conn_01x05_Pin, J7 Conn_ARM_JTAG_SWD_10, SW1 SW_Push, SW2 SW_Push, U1 STM32H753IITx, U2 ST1S40IDR, U3 TPS2121RUX, U4 USB3300-EZK, U5 MCP2562-E-SN, U6 W25Q128JVS, Y1 SG-210STF, Y2 8MHz, Y3 Crystal

Commit message: pf13, pf14, pf15, pg0, add qspi to readme
Connections:
- J2 pad 57: unconnected-(J2-Pin_57-Pad57) -> /PF15
- J2 pad 58: unconnected-(J2-Pin_58-Pad58) -> /PG0
- J2 pad 59: unconnected-(J2-Pin_59-Pad59) -> /PF13
- J2 pad 60: unconnected-(J2-Pin_60-Pad60) -> /PF14
- U1 pad 63: unconnected-(U1-PF13-Pad63) -> /PF13
- U1 pad 64: unconnected-(U1-PF14-Pad64) -> /PF14
- U1 pad 65: unconnected-(U1-PF15-Pad65) -> /PF15
- U1 pad 66: unconnected-(U1-PG0-Pad66) -> /PG0
Routing:
- net /PF13: track 0.00 -> 33.6 mm, vias 0 -> 1
- net /PF15: track 0.00 -> 29.9 mm, vias 0 -> 1
- net /PF14: track 0.00 -> 24.4 mm, vias 0 -> 1
- net /PG0: track 0.00 -> 24.4 mm, vias 0 -> 1
- net GND: vias 104 -> 103

Commit message: change all references from 753 to 743
Parts:
- U1: value STM32H753IITx -> STM32H743IITx
Other:
- board text added: "STM32H743 USB-HS CANbus Dev Board"
- board text removed: "STM32H753 USB-HS CANbus Dev Board"

Commit message: more io routing, pinion experimentation
Parts:
- moved J2 14.1 mm to (189.5, 123.8)
- moved C1 14.1 mm to (146.4, 83.4)
- moved C10 14.1 mm to (150.7, 108.1)
- moved C11 14.1 mm to (150.7, 100.9)
- moved C12 14.1 mm to (151.2, 89.4)
- moved C13 14.1 mm to (144.9, 111.9)
- moved C14 14.1 mm to (121.8, 97.9)
- moved C15 14.1 mm to (178.1, 96.8)
- moved C16 14.1 mm to (178.1, 98.3)
- moved C17 14.1 mm to (170.2, 100.2)
- moved C18 14.1 mm to (172.5, 100.7)
- moved C19 14.1 mm to (180.9, 90.3)
- moved C2 14.1 mm to (139.2, 83.0)
- moved C20 14.1 mm to (183.9, 97.4)
- moved C21 14.1 mm to (177.7, 93.7)
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Connections:
- J2 pad 41: unconnected-(J2-Pin_41-Pad41) -> /PH10
- J2 pad 42: unconnected-(J2-Pin_42-Pad42) -> /PH11
- J2 pad 43: unconnected-(J2-Pin_43-Pad43) -> /PH8
- J2 pad 44: unconnected-(J2-Pin_44-Pad44) -> /PH9
- J2 pad 45: unconnected-(J2-Pin_45-Pad45) -> /PH6
- J2 pad 46: unconnected-(J2-Pin_46-Pad46) -> /PH7
- J2 pad 47: unconnected-(J2-Pin_47-Pad47) -> /PE14
- J2 pad 48: unconnected-(J2-Pin_48-Pad48) -> /PE15
- J2 pad 49: unconnected-(J2-Pin_49-Pad49) -> /PE12
- J2 pad 50: unconnected-(J2-Pin_50-Pad50) -> /PE13
- J2 pad 51: unconnected-(J2-Pin_51-Pad51) -> /PE10
- J2 pad 52: unconnected-(J2-Pin_52-Pad52) -> /PE11
- J2 pad 53: unconnected-(J2-Pin_53-Pad53) -> /PE8
- J2 pad 54: unconnected-(J2-Pin_54-Pad54) -> /PE9
- J2 pad 55: unconnected-(J2-Pin_55-Pad55) -> /PG1
- J2 pad 56: unconnected-(J2-Pin_56-Pad56) -> /PE7
- U1 pad 67: unconnected-(U1-PG1-Pad67) -> /PG1
- U1 pad 68: unconnected-(U1-PE7-Pad68) -> /PE7
- U1 pad 69: unconnected-(U1-PE8-Pad69) -> /PE8
- U1 pad 70: unconnected-(U1-PE9-Pad70) -> /PE9
- U1 pad 73: unconnected-(U1-PE10-Pad73) -> /PE10
- U1 pad 74: unconnected-(U1-PE11-Pad74) -> /PE11
- U1 pad 75: unconnected-(U1-PE12-Pad75) -> /PE12
- U1 pad 76: unconnected-(U1-PE13-Pad76) -> /PE13
- U1 pad 77: unconnected-(U1-PE14-Pad77) -> /PE14
- U1 pad 78: unconnected-(U1-PE15-Pad78) -> /PE15
- U1 pad 83: unconnected-(U1-PH6-Pad83) -> /PH6
- U1 pad 84: unconnected-(U1-PH7-Pad84) -> /PH7
- U1 pad 85: unconnected-(U1-PH8-Pad85) -> /PH8
- U1 pad 86: unconnected-(U1-PH9-Pad86) -> /PH9
- U1 pad 87: unconnected-(U1-PH10-Pad87) -> /PH10
- U1 pad 88: unconnected-(U1-PH11-Pad88) -> /PH11
Routing:
- net /PG1: track 0.00 -> 29.5 mm, vias 0 -> 1
- net /PE8: track 0.00 -> 27.6 mm, vias 0 -> 1
- net /PE10: track 0.00 -> 24.1 mm, vias 0 -> 1
- net /PE7: track 0.00 -> 23.8 mm, vias 0 -> 1
- net /PE11: track 0.00 -> 23.2 mm, vias 0 -> 1
- net /PH6: track 0.00 -> 23.0 mm, vias 0 -> 1
- net /PE12: track 0.00 -> 22.4 mm, vias 0 -> 1
- net /PE9: track 0.00 -> 22.2 mm, vias 0 -> 1
- net /PE13: track 0.00 -> 21.6 mm, vias 0 -> 1
- net /PE14: track 0.00 -> 21.1 mm, vias 0 -> 1
- net /PH10: track 0.00 -> 20.6 mm, vias 0 -> 1
- net /PH8: track 0.00 -> 20.5 mm, vias 0 -> 1
- net /PH7: track 0.00 -> 20.0 mm, vias 0 -> 1
- net /PE15: track 0.00 -> 19.5 mm, vias 0 -> 1
- net /PH9: track 0.00 -> 17.6 mm, vias 0 -> 1
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
Commit message: rgb led, route io
Parts:
- added D3: LED_RGB, LED_SMD:LED_RGB_Wuerth-PLCC4_3.2x2.8mm_150141M173100, F.Cu at (185.9, 116.2)
- added Q1: BSS138, Package_TO_SOT_SMD:SOT-323_SC-70, F.Cu at (180.4, 112.3)
- added Q2: BSS138, Package_TO_SOT_SMD:SOT-323_SC-70, F.Cu at (180.4, 114.7)
- added Q3: BSS138, Package_TO_SOT_SMD:SOT-323_SC-70, F.Cu at (180.4, 117.1)
- added R21: 5.1R, Resistor_SMD:R_0402_1005Metric, F.Cu at (183.0, 116.0)
- added R22: 5.1R, Resistor_SMD:R_0402_1005Metric, F.Cu at (183.0, 114.9)
- added R23: 68R, Resistor_SMD:R_0402_1005Metric, F.Cu at (183.0, 117.1)
- added R24: 1k, Resistor_SMD:R_0402_1005Metric, F.Cu at (178.4, 112.3)
- added R25: 1k, Resistor_SMD:R_0402_1005Metric, F.Cu at (178.4, 114.8)
- added R26: 1k, Resistor_SMD:R_0402_1005Metric, F.Cu at (178.4, 117.1)
- moved TP2 4.40 mm to (157.8, 96.7)
- moved C11 0.78 mm to (151.1, 101.5), turned to 0 degrees
- moved C31 0.53 mm to (151.2, 95.9), turned to 0 degrees
Connections:
- J1 pad 60: unconnected-(J1-Pin_60-Pad60) -> GND
- J1 pad 62: unconnected-(J1-Pin_62-Pad62) -> GND
- J1 pad 64: unconnected-(J1-Pin_64-Pad64) -> GND
- J2 pad 10: unconnected-(J2-Pin_10-Pad10) -> GND
- J2 pad 11: unconnected-(J2-Pin_11-Pad11) -> GND
- J2 pad 12: unconnected-(J2-Pin_12-Pad12) -> GND
- J2 pad 13: unconnected-(J2-Pin_13-Pad13) -> /PI0
- J2 pad 14: unconnected-(J2-Pin_14-Pad14) -> /PI1
- J2 pad 15: unconnected-(J2-Pin_15-Pad15) -> /PH14
- J2 pad 16: unconnected-(J2-Pin_16-Pad16) -> /PH15
- J2 pad 17: unconnected-(J2-Pin_17-Pad17) -> /PA9
- J2 pad 18: unconnected-(J2-Pin_18-Pad18) -> /PA10
- J2 pad 19: unconnected-(J2-Pin_19-Pad19) -> /PA8
- J2 pad 20: unconnected-(J2-Pin_20-Pad20) -> /PC9
- J2 pad 21: unconnected-(J2-Pin_21-Pad21) -> /PC7
- J2 pad 22: unconnected-(J2-Pin_22-Pad22) -> /PC8
- J2 pad 23: unconnected-(J2-Pin_23-Pad23) -> /PG8
- J2 pad 24: unconnected-(J2-Pin_24-Pad24) -> /PC6
- J2 pad 25: unconnected-(J2-Pin_25-Pad25) -> /PG5
- J2 pad 26: unconnected-(J2-Pin_26-Pad26) -> /PG7
- J2 pad 27: unconnected-(J2-Pin_27-Pad27) -> /PG3
- J2 pad 28: unconnected-(J2-Pin_28-Pad28) -> /PG4
- J2 pad 29: unconnected-(J2-Pin_29-Pad29) -> /PD15
- J2 pad 30: unconnected-(J2-Pin_30-Pad30) -> /PG2
- J2 pad 31: unconnected-(J2-Pin_31-Pad31) -> /PD13
- J2 pad 32: unconnected-(J2-Pin_32-Pad32) -> /PD14
- J2 pad 33: unconnected-(J2-Pin_33-Pad33) -> /PD11
- J2 pad 34: unconnected-(J2-Pin_34-Pad34) -> /PD12
- J2 pad 35: unconnected-(J2-Pin_35-Pad35) -> /PD9
- J2 pad 36: unconnected-(J2-Pin_36-Pad36) -> /PD10
- J2 pad 37: unconnected-(J2-Pin_37-Pad37) -> /PB15
- J2 pad 38: unconnected-(J2-Pin_38-Pad38) -> /PD8
- J2 pad 39: unconnected-(J2-Pin_39-Pad39) -> /PH12
- J2 pad 40: unconnected-(J2-Pin_40-Pad40) -> /PB14
- J2 pad 5: unconnected-(J2-Pin_5-Pad5) -> +3V3
- J2 pad 6: unconnected-(J2-Pin_6-Pad6) -> +3V3
- J2 pad 7: unconnected-(J2-Pin_7-Pad7) -> GND
- J2 pad 8: unconnected-(J2-Pin_8-Pad8) -> GND
- J2 pad 9: unconnected-(J2-Pin_9-Pad9) -> GND
- U1 pad 100: unconnected-(U1-PD12-Pad100) -> /PD12
- U1 pad 101: unconnected-(U1-PD13-Pad101) -> /PD13
- U1 pad 104: unconnected-(U1-PD14-Pad104) -> /PD14
- U1 pad 105: unconnected-(U1-PD15-Pad105) -> /PD15
- U1 pad 106: unconnected-(U1-PG2-Pad106) -> /PG2
- U1 pad 107: unconnected-(U1-PG3-Pad107) -> /PG3
- U1 pad 108: unconnected-(U1-PG4-Pad108) -> /PG4
- U1 pad 109: unconnected-(U1-PG5-Pad109) -> /PG5
- U1 pad 111: unconnected-(U1-PG7-Pad111) -> /PG7
- U1 pad 112: unconnected-(U1-PG8-Pad112) -> /PG8
- U1 pad 115: unconnected-(U1-PC6-Pad115) -> /PC6
- U1 pad 116: unconnected-(U1-PC7-Pad116) -> /PC7
- U1 pad 117: unconnected-(U1-PC8-Pad117) -> /PC8
- U1 pad 118: unconnected-(U1-PC9-Pad118) -> /PC9
- U1 pad 119: unconnected-(U1-PA8-Pad119) -> /PA8
- U1 pad 120: unconnected-(U1-PA9-Pad120) -> /PA9
- U1 pad 121: unconnected-(U1-PA10-Pad121) -> /PA10
- U1 pad 129: unconnected-(U1-PH14-Pad129) -> /PH14
- U1 pad 130: unconnected-(U1-PH15-Pad130) -> /PH15
- U1 pad 89: unconnected-(U1-PH12-Pad89) -> /PH12
- U1 pad 94: unconnected-(U1-PB14-Pad94) -> /PB14
- U1 pad 95: unconnected-(U1-PB15-Pad95) -> /PB15
- U1 pad 96: unconnected-(U1-PD8-Pad96) -> /PD8
- U1 pad 97: unconnected-(U1-PD9-Pad97) -> /PD9
- U1 pad 98: unconnected-(U1-PD10-Pad98) -> /PD10
- U1 pad 99: unconnected-(U1-PD11-Pad99) -> /PD11
Routing:
- net /PI0: track 0.00 -> 59.2 mm, vias 0 -> 1
- net /PI1: track 0.00 -> 54.9 mm, vias 0 -> 1
- net /PA9: track 0.00 -> 52.2 mm, vias 0 -> 1
- net /PA8: track 0.00 -> 51.8 mm, vias 0 -> 1
- net /PH14: track 0.00 -> 51.4 mm, vias 0 -> 1
- net /PH15: track 0.00 -> 49.4 mm, vias 0 -> 1
- net /PC7: track 0.00 -> 49.1 mm, vias 0 -> 1
- net /PA10: track 0.00 -> 48.9 mm, vias 0 -> 1
- net /PC9: track 0.00 -> 46.4 mm, vias 0 -> 1
- net /PC8: track 0.00 -> 46.3 mm, vias 0 -> 1
- net /PC6: track 0.00 -> 45.7 mm, vias 0 -> 1
- net /PG8: track 0.00 -> 34.5 mm, vias 0 -> 1
- net /PG5: track 0.00 -> 32.3 mm, vias 0 -> 1
- net /PG7: track 0.00 -> 30.2 mm, vias 0 -> 1
- net /PG3: track 0.00 -> 29.2 mm, vias 0 -> 1
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Other:
- board text added: "Design by Kevin Ahr kevinbot.net/h743-can-hs"
- board text removed: "Design by Kevin Ahr kevinbot.net"
