File: stm32h753_dev.kicad_pcb (KiCad board)
At the start: 4 copper layers, 99.1 x 53.3 mm, 100 parts, among them J1 Conn_02x38_Counter_Clockwise, J2 Conn_02x38_Counter_Clockwise, J3 USB_C_Receptacle_USB2.0_16P, J4 USB_C_Receptacle_USB2.0_16P, J5 DE9_Pins_MountingHoles, J6 Conn_01x05_Pin, J7 Conn_ARM_JTAG_SWD_10, Q1 BSS138, Q2 BSS138, Q3 BSS138, SW1 SW_Push, SW2 SW_Push, U1 STM32H743IITx, U2 ST1S40IDR, U3 TPS2121RUX, U4 USB3300-EZK, U5 MCP2562-E-SN, U6 W25Q128JVS, Y1 SG-210STF, Y2 8MHz, Y3 Crystal

Commit message: rgb gates, pinion changes
Parts:
- J5: value DE9_Pins_MountingHoles -> DE9_Pins_MH
Connections:
- R24 pad 1: unconnected-(R24-Pad1) -> /PC8
- R25 pad 1: unconnected-(R25-Pad1) -> /PA7
- R26 pad 1: unconnected-(R26-Pad1) -> /PA6
Routing:
- net /PA7: track 33.7 -> 113.1 mm
- net /PA6: track 32.8 -> 107.0 mm
- net /PC8: track 46.3 -> 70.9 mm
- net Net-(Q2-G): track 0.00 -> 1.21 mm
- net Net-(Q1-G): track 0.00 -> 1.18 mm
- net Net-(Q3-G): track 0.00 -> 1.17 mm

Commit message: power led
Parts:
- added D4: LED, LED_SMD:LED_0603_1608Metric, F.Cu at (189.7, 81.7)
- added R27: 300R, Resistor_SMD:R_0402_1005Metric, F.Cu at (187.6, 81.5)
Routing:
- net Net-(D4-A): track 0.00 -> 1.44 mm
- net VBUS: track 139.8 -> 140.5 mm
Other:
- board text added: "Power"
