File: stm32h743_can_hs.kicad_pcb (KiCad board)
At the start: 4 copper layers, 99.1 x 53.3 mm, 102 parts, among them J1 Conn_02x38_Counter_Clockwise, J2 Conn_02x38_Counter_Clockwise, J3 USB_C_Receptacle_USB2.0_16P, J4 USB_C_Receptacle_USB2.0_16P, J5 DE9_Pins_MH, J6 Conn_01x05_Pin, J7 Conn_ARM_JTAG_SWD_10, Q1 BSS138, Q2 BSS138, Q3 BSS138, SW1 SW_Push, SW2 SW_Push, U1 STM32H743IITx, U2 ST1S40IDR, U3 TPS2121RUX, U4 USB3300-EZK, U5 MCP2562-E-SN, U6 W25Q128JVS, Y1 SG-210STF, Y2 8MHz, Y3 Crystal

Commit message: bom changes
Parts:
- U6: value W25Q128JVS -> S25FL128LAGMFI013
Routing:
- net GND: vias 184 -> 210
Changed lines of the file:
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@@
 			)
 		)
-		(property "Part Number" "RC0402FR-07300RL"
+		(property "Part Number" "RC0402JR-07300RL"
 			(at 0 0 90)
 			(unlocked yes)
@@
 			)
 		)
-		(property "Part Number" "RC0402FR-0775KL"
+		(property "Part Number" "RC0402JR-0775KL"
 			(at 0 0 270)
 			(unlocked yes)
@@
 			)
 		)
-		(property "Value" "W25Q128JVS"
+		(property "Value" "S25FL128LAGMFI013"
 			(at 0 3.6 0)
 			(layer "F.Fab")
@@
 			)
 		)
-		(property "Part Number" "W25Q128JVSIQ TR"
+		(property "Part Number" "S25FL128LAGMFI013"
 			(at 0 0 0)
 			(unlocked yes)
@@
 			(net "GND")
 			(pinfunction "ST_9")
-			(pintype "open_collector")
+			(pintype "passive")
 		)
 		(pad "10" smd roundrect
@@
 	)
 	(via
+		(at 178.8 89.2)
+		(size 0.6)
+		(drill 0.3)
+		(layers "F.Cu" "B.Cu")
+		(free yes)
+		(net "GND")
+	)
+	(via
+		(at 174.7 107.9)
+		(size 0.6)
+		(drill 0.3)
+		(layers "F.Cu" "B.Cu")
+		(free yes)
+		(net "GND")
+	)
+	(via
 		(at 122.8 109.7)
 		(size 0.6)
@@
 	)
 	(via
+		(at 132.5 89)
+		(size 0.6)
+		(drill 0.3)
+		(layers "F.Cu" "B.Cu")
+		(free yes)
+		(net "GND")
+	)
+	(via
 		(at 125.162188 97.558126)
 		(size 0.6)
@@
 	)
 	(via
+		(at 113.5 107.7)
+		(size 0.6)
+		(drill 0.3)
+		(layers "F.Cu" "B.Cu")
+		(free yes)
+		(net "GND")
+	)
+	(via
 		(at 180.5 101.6)
 		(size 0.6)
@@
 	)
 	(via
+		(at 169.7 101.6)
+		(size 0.6)
+		(drill 0.3)
+		(layers "F.Cu" "B.Cu")
+		(free yes)
+		(net "GND")
+	)
+	(via
 		(at 187.4 104.6)
 		(size 0.6)
@@
 	)
 	(via
+		(at 111.3 106.5)
+		(size 0.6)
+		(drill 0.3)
+		(layers "F.Cu" "B.Cu")
+		(free yes)
+		(net "GND")
+	)
+	(via
+		(at 121.5 96.2)
+		(size 0.6)
+		(drill 0.3)
+		(layers "F.Cu" "B.Cu")
+		(free yes)
+		(net "GND")
+	)
+	(via
 		(at 127.2 90.8)
 		(size 0.6)
@@
 	)
 	(via
+		(at 155.7 107.3)
+		(size 0.6)
+		(drill 0.3)
+		(layers "F.Cu" "B.Cu")
+		(free yes)
+		(net "GND")
+	)
+	(via
 		(at 145.7 119.5)
 		(size 0.6)
@@
 	)
 	(via
+		(at 143.5 88.9)
+		(size 0.6)
+		(drill 0.3)
+		(layers "F.Cu" "B.Cu")
+		(free yes)
+		(net "GND")
+	)
+	(via
 		(at 134.551094 86.120768)
 		(size 0.6)
@@
 	)
 	(via
+		(at 138.3 98.1)
+		(size 0.6)
+		(drill 0.3)
+		(layers "F.Cu" "B.Cu")
+		(free yes)
+		(net "GND")
+	)
+	(via
 		(at 161.855 94.51625)
 		(size 0.6)
@@
 	)
 	(via
+		(at 185.8 116.6)
+		(size 0.6)
+		(drill 0.3)
+		(layers "F.Cu" "B.Cu")
+		(free yes)
+		(net "GND")
+	)
+	(via
+		(at 140.3 98.8)
+		(size 0.6)
+		(drill 0.3)
+		(layers "F.Cu" "B.Cu")
+		(free yes)
+		(net "GND")
+	)
+	(via
 		(at 144.4 119.5)
 		(size 0.6)
@@
 	)
 	(via
+		(at 135.2 96)
+		(size 0.6)
+		(drill 0.3)
+		(layers "F.Cu" "B.Cu")
+		(free yes)
+		(net "GND")
+	)
+	(via
 		(at 179.1 103.15)
 		(size 0.6)
@@
 	)
 	(via
+		(at 135 83.8)
+		(size 0.6)
+		(drill 0.3)
+		(layers "F.Cu" "B.Cu")
+		(free yes)
+		(net "GND")
+	)
+	(via
 		(at 143.1 108.6)
 		(size 0.6)
@@
 	)
 	(via
+		(at 165 105.5)
+		(size 0.6)
+		(drill 0.3)
+		(layers "F.Cu" "B.Cu")
+		(free yes)
+		(net "GND")
+	)
+	(via
 		(at 138.3 107)
 		(size 0.6)
@@
 	)
 	(via
+		(at 186.7 82.8)
+		(size 0.6)
+		(drill 0.3)
+		(layers "F.Cu" "B.Cu")
+		(free yes)
+		(net "GND")
+	)
+	(via
 		(at 148.077836 101.913126)
 		(size 0.6)
@@
 	)
 	(via
+		(at 175.3 87.2)
+		(size 0.6)
+		(drill 0.3)
+		(layers "F.Cu" "B.Cu")
+		(free yes)
+		(net "GND")
+	)
+	(via
 		(at 182.2 109.2)
 		(size 0.6)
@@
 	)
 	(via
+		(at 176.9 117.3)
+		(size 0.6)
+		(drill 0.3)
+		(layers "F.Cu" "B.Cu")
+		(free yes)
+		(net "GND")
+	)
+	(via
 		(at 111.2 92.8)
 		(size 0.6)
@@
 	)
 	(via
+		(at 151.7 85.9)
+		(size 0.6)
+		(drill 0.3)
+		(layers "F.Cu" "B.Cu")
+		(free yes)
+		(net "GND")
+	)
+	(via
 		(at 161.805 104.3325)
 		(size 0.6)
@@
 	)
 	(via
+		(at 135.1 88.9)
+		(size 0.6)
+		(drill 0.3)
+		(layers "F.Cu" "B.Cu")
+		(free yes)
+		(net "GND")
+	)
+	(via
 		(at 107.5 94.468675)
 		(size 0.6)
@@
 	)
 	(via
+		(at 174.2 92.6)
+		(size 0.6)
+		(drill 0.3)
+		(layers "F.Cu" "B.Cu")
+		(free yes)
+		(net "GND")
+	)
+	(via
 		(at 172.3 109.9)
 		(size 0.6)
@@
 	)
 	(via
+		(at 157.7 107.8)
+		(size 0.6)
+		(drill 0.3)
+		(layers "F.Cu" "B.Cu")
+		(free yes)
+		(net "GND")
+	)
+	(via
 		(at 131.6 108.8)
 		(size 0.6)
@@
 	)
 	(via
+		(at 168.5 111.9)
+		(size 0.6)
+		(drill 0.3)
+		(layers "F.Cu" "B.Cu")
+		(free yes)
+		(net "GND")
+	)
+	(via
 		(at 103.1 89.4)
 		(size 0.6)
@@
 	)
 	(via
+		(at 132.9 95.4)
+		(size 0.6)
+		(drill 0.3)
+		(layers "F.Cu" "B.Cu")
+		(free yes)
+		(net "GND")
+	)
+	(via
 		(at 125.462188 93.658126)
 		(size 0.6)
@@
 		(net "GND")
 	)
+	(via
+		(at 133.9 98.3)
+		(size 0.6)
+		(drill 0.3)
+		(layers "F.Cu" "B.Cu")
+		(free yes)
+		(net "GND")
+	)
+	(via
+		(at 158.2 109.8)
+		(size 0.6)
+		(drill 0.3)
+		(layers "F.Cu" "B.Cu")
+		(free yes)
+		(net "GND")
+	)

Commit message: cleanup, board rev
Routing:
- net /PA9: track 52.2 -> 51.6 mm
- net GND: vias 210 -> 216
Changed lines of the file:
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@@
 	)
 	(via
+		(at 145.7 93.1)
+		(size 0.6)
+		(drill 0.3)
+		(layers "F.Cu" "B.Cu")
+		(free yes)
+		(net "GND")
+	)
+	(via
 		(at 132.5 89)
 		(size 0.6)
@@
 	)
 	(via
+		(at 142.7 93.1)
+		(size 0.6)
+		(drill 0.3)
+		(layers "F.Cu" "B.Cu")
+		(free yes)
+		(net "GND")
+	)
+	(via
 		(at 117.8 107)
 		(size 0.6)
@@
 	)
 	(via
+		(at 140 95.6)
+		(size 0.6)
+		(drill 0.3)
+		(layers "F.Cu" "B.Cu")
+		(free yes)
+		(net "GND")
+	)
+	(via
 		(at 174.15 98.9)
 		(size 0.6)
@@
 	)
 	(via
+		(at 155.2 95.2)
+		(size 0.6)
+		(drill 0.3)
+		(layers "F.Cu" "B.Cu")
+		(free yes)
+		(net "GND")
+	)
+	(via
 		(at 129.5 103.4)
 		(size 0.6)
@@
 	)
 	(via
+		(at 145.7 95.6)
+		(size 0.6)
+		(drill 0.3)
+		(layers "F.Cu" "B.Cu")
+		(free yes)
+		(net "GND")
+	)
+	(via
 		(at 119.267603 101.913541)
 		(size 0.6)
@@
 	)
 	(via
+		(at 142.7 95.6)
+		(size 0.6)
+		(drill 0.3)
+		(layers "F.Cu" "B.Cu")
+		(free yes)
+		(net "GND")
+	)
+	(via
 		(at 151.5 109.164594)
 		(size 0.6)
@@
 	)
 	(segment
-		(start 147.1 92.9)
-		(end 147.8 92.9)
+		(start 163 93.5)
+		(end 165.9 96.4)
 		(width 0.2)
 		(layer "In2.Cu")
@@
 	)
 	(segment
-		(start 147.8 92.9)
-		(end 149.9 95)
+		(start 165.9 117.8)
+		(end 165.5 118.2)
 		(width 0.2)
 		(layer "In2.Cu")
@@
 	)
 	(segment
-		(start 163 93.5)
-		(end 165.9 96.4)
+		(start 147.1 92.9)
+		(end 147.73842 92.9)
 		(width 0.2)
 		(layer "In2.Cu")
@@
 	)
 	(segment
-		(start 165.5 118.2)
-		(end 165.5 122.62)
+		(start 165.9 96.4)
+		(end 165.9 117.8)
 		(width 0.2)
 		(layer "In2.Cu")
@@
 	)
 	(segment
-		(start 149.9 95)
-		(end 156.800001 95)
+		(start 158.300001 93.5)
+		(end 163 93.5)
 		(width 0.2)
 		(layer "In2.Cu")
@@
 	)
 	(segment
-		(start 165.9 117.8)
-		(end 165.5 118.2)
+		(start 153.7 94.6)
+		(end 157.200001 94.6)
 		(width 0.2)
 		(layer "In2.Cu")
@@
 	)
 	(segment
-		(start 165.9 96.4)
-		(end 165.9 117.8)
+		(start 165.5 118.2)
+		(end 165.5 122.62)
 		(width 0.2)
 		(layer "In2.Cu")
@@
 	)
 	(segment
-		(start 158.300001 93.5)
-		(end 163 93.5)
+		(start 148.73842 91.9)
+		(end 151 91.9)
+		(width 0.2)
+		(layer "In2.Cu")
+		(net "/PA8")
+	)
+	(segment
+		(start 151 91.9)
+		(end 153.7 94.6)
 		(width 0.2)
 		(layer "In2.Cu")
@@
 	)
 	(segment
-		(start 156.800001 95)
+		(start 147.73842 92.9)
+		(end 148.73842 91.9)
+		(width 0.2)
+		(layer "In2.Cu")
+		(net "/PA8")
+	)
+	(segment
+		(start 157.200001 94.6)
 		(end 158.300001 93.5)
 		(width 0.2)
@@
 	)
 	(segment
-		(start 167.9 119.94)
-		(end 167.9 122.48)
+		(start 147.85 92.293446)
+		(end 148.593446 91.55)
 		(width 0.2)
 		(layer "In2.Cu")
@@
 	)
 	(segment
-		(start 147.541131 92.293446)
-		(end 147.688421 92.293446)
+		(start 167.9 119.94)
+		(end 167.9 122.48)
 		(width 0.2)
 		(layer "In2.Cu")
@@
 	)
 	(segment
-		(start 166.25 96.255026)
-		(end 166.25 118.29)
+		(start 148.593446 91.55)
+		(end 153.555026 91.55)
 		(width 0.2)
 		(layer "In2.Cu")
@@
 	)
 	(segment
-		(start 166.25 118.29)
-		(end 167.9 119.94)
+		(start 153.555026 91.55)
+		(end 155.155026 93.15)
 		(width 0.2)
 		(layer "In2.Cu")
@@
 	)
 	(segment
-		(start 156.655026 94.65)
-		(end 158.155027 93.15)
+		(start 155.155026 93.15)
+		(end 163.144974 93.15)
 		(width 0.2)
 		(layer "In2.Cu")
@@
 	)
 	(segment
-		(start 150.044974 94.65)
-		(end 156.655026 94.65)
+		(start 163.144974 93.15)
+		(end 166.25 96.255026)
 		(width 0.2)
 		(layer "In2.Cu")
@@
 	)
 	(segment
-		(start 163.144974 93.15)
-		(end 166.25 96.255026)
+		(start 166.25 96.255026)
+		(end 166.25 118.29)
 		(width 0.2)
 		(layer "In2.Cu")
@@
 	)
 	(segment
-		(start 147.688421 92.293446)
-		(end 150.044974 94.65)
+		(start 166.25 118.29)
+		(end 167.9 119.94)
 		(width 0.2)
 		(layer "In2.Cu")
@@
 	)
 	(segment
-		(start 158.155027 93.15)
-		(end 163.144974 93.15)
+		(start 147.541131 92.293446)
+		(end 147.85 92.293446)
 		(width 0.2)
 		(layer "In2.Cu")
@@
 	)
 	(segment
-		(start 166.6 118.1)
-		(end 169.22 120.72)
+		(start 148.071002 91.2)
+		(end 153.7 91.2)
 		(width 0.2)
 		(layer "In2.Cu")
@@
 	)
 	(segment
-		(start 154.7 92.8)
-		(end 163.289948 92.8)
+		(start 166.6 118.1)
+		(end 169.22 120.72)
 		(width 0.2)
 		(layer "In2.Cu")
@@
 	)
 	(segment
-		(start 147.708618 91.562384)
-		(end 147.946234 91.8)
+		(start 166.6 96.110052)
+		(end 166.6 118.1)
 		(width 0.2)
 		(layer "In2.Cu")
@@
 	)
 	(segment
-		(start 153.7 91.8)
-		(end 154.7 92.8)
+		(start 169.22 120.72)
+		(end 169.22 121.26)
 		(width 0.2)
 		(layer "In2.Cu")
@@
 	)
 	(segment
-		(start 169.22 120.72)
-		(end 169.22 121.26)
+		(start 147.708618 91.562384)
+		(end 148.071002 91.2)
 		(width 0.2)
 		(layer "In2.Cu")
@@
 	)
 	(segment
-		(start 166.6 96.110052)
-		(end 166.6 118.1)
+		(start 155.3 92.8)
+		(end 163.289948 92.8)
 		(width 0.2)
 		(layer "In2.Cu")
@@
 	)
 	(segment
-		(start 147.946234 91.8)
-		(end 153.7 91.8)
+		(start 153.7 91.2)
+		(end 155.3 92.8)
 		(width 0.2)
 		(layer "In2.Cu")

Commit message: fix field warnings, erc, drc, vias
Parts:
- R1: value 75k -> 75k 1%
- R10, R11, R2: value 24k -> 24k 1%
- R19, R20: value 60.4R -> 60.4R 1%
Routing:
- net GND: vias 216 -> 234
