File: stm32h743_can_hs.kicad_pcb (KiCad board)
At the start: 4 copper layers, 99.1 x 53.3 mm, 102 parts, among them J1 Conn_02x38_Counter_Clockwise, J2 Conn_02x38_Counter_Clockwise, J3 USB_C_Receptacle_USB2.0_16P, J4 USB_C_Receptacle_USB2.0_16P, J5 DE9_Pins_MH, J6 Conn_01x05_Pin, J7 Conn_ARM_JTAG_SWD_10, Q1 BSS138, Q2 BSS138, Q3 BSS138, SW1 SW_Push, SW2 SW_Push, U1 STM32H743IITx, U2 ST1S40IDR, U3 TPS2121RUX, U4 USB3300-EZK, U5 TCAN1044AVDRQ1, U6 S25FL128LAGMFI013, Y1 SG-210STF, Y2 8MHz, Y3 Crystal

Commit message: changes for production, fix cad models
Routing:
- net /PA6: track 109.5 -> 110.9 mm
- net GND: track 93.3 -> 93.4 mm, vias 252 -> 251

Commit message: fix buck ic part numbers
Parts:
- U2: value ST1S40IDR -> ST1S40IPHR
Changed lines of the file:
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@@
 		(capping no)
 		(filling no)
-		(zone_defaults)
 		(pcbplotparams
 			(layerselection 0x00000000_00000000_55ffffdf_ffffffff)
@@
 			)
 		)
-		(property "Value" "ST1S40IDR"
+		(property "Value" "ST1S40IPHR"
 			(at 4.7 5.39 90)
 			(layer "F.Fab")
@@
 			)
 		)
-		(property "manf#" "ST1S40IDR"
+		(property "manf#" "ST1S40IPHR"
 			(at 0 0 90)
 			(unlocked yes)
