File: stm32h743_can_hs.kicad_sch (KiCad schematic)
At the start: 100 parts, among them J1 Conn_02x38_Counter_Clockwise, J2 Conn_02x38_Counter_Clockwise, J3 USB_C_Receptacle_USB2.0_16P, J4 USB_C_Receptacle_USB2.0_16P, J5 DE9_Pins_MH, J6 Conn_01x05_Pin, J7 Conn_ARM_JTAG_SWD_10, Q1 BSS138, Q2 BSS138, Q3 BSS138, SW1 SW_Push, SW2 SW_Push, U1 STM32H743IITx, U2 ST1S40IPHR, U3 TPS2121RUX, U4 USB3300-EZK, U5 TCAN1044AVDRQ1, U6 S25FL128LAGMFI013, Y1 SG-210STF, Y2 8MHz, Y3 Crystal

Commit message: minor pcb cleanup, fixed bom
Parts:
- Q1, Q2, Q3: manf_alt1# (none) -> 2V7002WT1G
Changed lines of the file:
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@@
 			)
 		)
+		(property "manf_alt1#" "2V7002WT1G"
+			(at 457.2 78.74 0)
+			(hide yes)
+			(show_name no)
+			(do_not_autoplace no)
+			(effects
+				(font
+					(size 1.27 1.27)
+				)
+			)
+		)
 		(pin "3"
 		)
@@
 			)
 		)
+		(property "manf_alt1#" "2V7002WT1G"
+			(at 468.63 100.33 0)
+			(hide yes)
+			(show_name no)
+			(do_not_autoplace no)
+			(effects
+				(font
+					(size 1.27 1.27)
+				)
+			)
+		)
 		(pin "3"
 		)
@@
 			(at 436.88 66.04 0)
 			(hide yes)
+			(show_name no)
+			(do_not_autoplace no)
+			(effects
+				(font
+					(size 1.27 1.27)
+				)
+			)
+		)
+		(property "manf_alt1#" "2V7002WT1G"
+			(at 436.88 66.04 0)
+			(hide yes)

Commit message: sch: fix led symbol
Parts:
- D3: symbol Device:LED_ARGB -> Device:LED_ABRG
Connections:
- net at R22.2: now also D3.3 (RK); no longer D3.4 (BK)
- net at R21.2: now also D3.4 (GK); no longer D3.3 (GK)
Other:
- moved on the sheet: Q1, Q3, R22, R23, R24, R26
Changed lines of the file:
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@@
 	)
 	(label "PC8"
-		(at 424.18 66.04 180)
+		(at 455.93 100.33 180)
 		(effects
 			(font
@@
 	)
 	(label "PA6"
-		(at 455.93 100.33 180)
+		(at 424.18 66.04 180)
 		(effects
 			(font
@@
 	(symbol
 		(lib_id "Device:R")
-		(at 459.74 100.33 90)
+		(at 427.99 66.04 90)
 		(unit 1)
 		(body_style 1)
@@
 		(fields_autoplaced yes)
 		(property "Reference" "R26"
-			(at 459.74 93.98 90)
+			(at 427.99 59.69 90)
 			(show_name no)
 			(do_not_autoplace no)
@@
 		)
 		(property "Value" "1k"
-			(at 459.74 96.52 90)
+			(at 427.99 62.23 90)
 			(show_name no)
 			(do_not_autoplace no)
@@
 		)
 		(property "Footprint" "Resistor_SMD:R_0402_1005Metric"
-			(at 459.74 102.108 90)
+			(at 427.99 67.818 90)
 			(hide yes)
 			(show_name no)
@@
 		)
 		(property "Datasheet" ""
-			(at 459.74 100.33 0)
+			(at 427.99 66.04 0)
 			(hide yes)
 			(show_name no)
@@
 		)
 		(property "Description" "Resistor"
-			(at 459.74 100.33 0)
+			(at 427.99 66.04 0)
 			(hide yes)
 			(show_name no)
@@
 		)
 		(property "manf#" "RC0402JR-071KL"
-			(at 459.74 100.33 90)
+			(at 427.99 66.04 90)
 			(hide yes)
 			(show_name no)
@@
 	(symbol
 		(lib_id "Transistor_FET:BSS138")
-		(at 468.63 100.33 0)
+		(at 436.88 66.04 0)
 		(unit 1)
 		(body_style 1)
@@
 		(dnp no)
 		(property "Reference" "Q3"
-			(at 473.71 99.06 0)
+			(at 441.96 64.77 0)
 			(show_name no)
 			(do_not_autoplace no)
@@
 		)
 		(property "Value" "BSS138"
-			(at 473.71 101.6 0)
+			(at 441.96 67.31 0)
 			(show_name no)
 			(do_not_autoplace no)
@@
 		)
 		(property "Footprint" "Package_TO_SOT_SMD:SOT-323_SC-70"
-			(at 473.71 102.235 0)
+			(at 441.96 67.945 0)
 			(hide yes)
 			(show_name no)
@@
 		)
 		(property "Datasheet" "https://www.onsemi.com/pub/Collateral/BSS138-D.PDF"
-			(at 473.71 104.14 0)
+			(at 441.96 69.85 0)
 			(hide yes)
 			(show_name no)
@@
 		)
 		(property "Description" "50V Vds, 0.22A Id, N-Channel MOSFET, SOT-323"
-			(at 468.63 100.33 0)
+			(at 436.88 66.04 0)
 			(hide yes)
 			(show_name no)
@@
 		)
 		(property "manf#" "BSS138PW,115"
-			(at 468.63 100.33 0)
+			(at 436.88 66.04 0)
 			(hide yes)
 			(show_name no)
@@
 		)
 		(property "manf_alt1#" "2V7002WT1G"
-			(at 468.63 100.33 0)
+			(at 436.88 66.04 0)
 			(hide yes)
 			(show_name no)
@@
 	(symbol
 		(lib_id "Device:R")
-		(at 443.23 60.96 90)
+		(at 474.98 50.8 90)
 		(unit 1)
 		(body_style 1)
@@
 		(fields_autoplaced yes)
 		(property "Reference" "R22"
-			(at 443.23 54.61 90)
+			(at 474.98 44.45 90)
 			(show_name no)
 			(do_not_autoplace no)
@@
 		)
 		(property "Value" "5.1R"
-			(at 443.23 57.15 90)
+			(at 474.98 46.99 90)
 			(show_name no)
 			(do_not_autoplace no)
@@
 		)
 		(property "Footprint" "Resistor_SMD:R_0402_1005Metric"
-			(at 443.23 62.738 90)
+			(at 474.98 52.578 90)
 			(hide yes)
 			(show_name no)
@@
 		)
 		(property "Datasheet" ""
-			(at 443.23 60.96 0)
+			(at 474.98 50.8 0)
 			(hide yes)
 			(show_name no)
@@
 		)
 		(property "Description" "Resistor"
-			(at 443.23 60.96 0)
+			(at 474.98 50.8 0)
 			(hide yes)
 			(show_name no)
@@
 		)
 		(property "manf#" "RC0402JR-075R1L"
-			(at 443.23 60.96 90)
+			(at 474.98 50.8 90)
 			(hide yes)
 			(show_name no)
@@
 	(symbol
 		(lib_id "Transistor_FET:BSS138")
-		(at 436.88 66.04 0)
+		(at 468.63 100.33 0)
 		(unit 1)
 		(body_style 1)
@@
 		(dnp no)
 		(property "Reference" "Q1"
-			(at 441.96 64.77 0)
+			(at 473.71 99.06 0)
 			(show_name no)
 			(do_not_autoplace no)
@@
 		)
 		(property "Value" "BSS138"
-			(at 441.96 67.31 0)
+			(at 473.71 101.6 0)
 			(show_name no)
 			(do_not_autoplace no)
@@
 		)
 		(property "Footprint" "Package_TO_SOT_SMD:SOT-323_SC-70"
-			(at 441.96 67.945 0)
+			(at 473.71 102.235 0)
 			(hide yes)
 			(show_name no)
@@
 		)
 		(property "Datasheet" "https://www.onsemi.com/pub/Collateral/BSS138-D.PDF"
-			(at 441.96 69.85 0)
+			(at 473.71 104.14 0)
 			(hide yes)
 			(show_name no)
@@
 		)
 		(property "Description" "50V Vds, 0.22A Id, N-Channel MOSFET, SOT-323"
-			(at 436.88 66.04 0)
+			(at 468.63 100.33 0)
 			(hide yes)
 			(show_name no)
@@
 		)
 		(property "manf#" "BSS138PW,115"
-			(at 436.88 66.04 0)
+			(at 468.63 100.33 0)
 			(hide yes)
 			(show_name no)
@@
 		)
 		(property "manf_alt1#" "2V7002WT1G"
-			(at 436.88 66.04 0)
+			(at 468.63 100.33 0)
 			(hide yes)
 			(show_name no)
@@
 	)
 	(symbol
-		(lib_id "Device:LED_ARGB")
+		(lib_id "Device:LED_ABRG")
 		(at 483.87 55.88 0)
 		(unit 1)
@@
 			)
 		)
-		(property "Description" "RGB LED, anode/red/green/blue"
+		(property "Description" "RGB LED, anode/blue/red/green"
 			(at 483.87 55.88 0)
 			(hide yes)
@@
 	(symbol
 		(lib_id "Device:R")
-		(at 474.98 50.8 90)
+		(at 443.23 60.96 90)
 		(unit 1)
 		(body_style 1)
@@
 		(fields_autoplaced yes)
 		(property "Reference" "R23"
-			(at 474.98 44.45 90)
+			(at 443.23 54.61 90)
 			(show_name no)
 			(do_not_autoplace no)
@@
 		)
 		(property "Value" "68R"
-			(at 474.98 46.99 90)
+			(at 443.23 57.15 90)
 			(show_name no)
 			(do_not_autoplace no)
@@
 		)
 		(property "Footprint" "Resistor_SMD:R_0402_1005Metric"
-			(at 474.98 52.578 90)
+			(at 443.23 62.738 90)
 			(hide yes)
 			(show_name no)
@@
 		)
 		(property "Datasheet" ""
-			(at 474.98 50.8 0)
+			(at 443.23 60.96 0)
 			(hide yes)
 			(show_name no)
@@
 		)
 		(property "Description" "Resistor"
-			(at 474.98 50.8 0)
+			(at 443.23 60.96 0)
 			(hide yes)
 			(show_name no)
@@
 		)
 		(property "manf#" "RC0402JR-0768RL"
-			(at 474.98 50.8 90)
+			(at 443.23 60.96 90)
 			(hide yes)
 			(show_name no)
@@
 	(symbol
 		(lib_id "Device:R")
-		(at 427.99 66.04 90)
+		(at 459.74 100.33 90)
 		(unit 1)
 		(body_style 1)
@@
 		(fields_autoplaced yes)
 		(property "Reference" "R24"
-			(at 427.99 59.69 90)
+			(at 459.74 93.98 90)
 			(show_name no)
 			(do_not_autoplace no)
@@
 		)
 		(property "Value" "1k"
-			(at 427.99 62.23 90)
+			(at 459.74 96.52 90)
 			(show_name no)
 			(do_not_autoplace no)
@@
 		)
 		(property "Footprint" "Resistor_SMD:R_0402_1005Metric"
-			(at 427.99 67.818 90)
+			(at 459.74 102.108 90)
 			(hide yes)
 			(show_name no)
@@
 		)
 		(property "Datasheet" ""
-			(at 427.99 66.04 0)
+			(at 459.74 100.33 0)
 			(hide yes)
 			(show_name no)
@@
 		)
 		(property "Description" "Resistor"
-			(at 427.99 66.04 0)
+			(at 459.74 100.33 0)
 			(hide yes)
 			(show_name no)
@@
 		)
 		(property "manf#" "RC0402JR-071KL"
-			(at 427.99 66.04 90)
+			(at 459.74 100.33 90)
 			(hide yes)
 			(show_name no)

Commit message: replace debug header with stdc14, add PA13 to I/O, split pinion/ibom between versions
Parts:
- removed J7: Conn_ARM_JTAG_SWD_10, FTSH-105-01-L-DV-K:SAMTEC_FTSH-105-01-L-DV-K, symbol Connector:Conn_ARM_JTAG_SWD_10
- added J7: Conn_ST_STDC14, SAMTEC_FTSH-107-01-X-DV-K:SAMTEC_FTSH-107-01-X-DV-K, symbol Connector:Conn_ST_STDC14
Connections:
- net +3V3: now also J7.3 (VCC)
- net GND: now also J7.11 (GNDDetect), J7.5 (GND), J7.7 (GND); no longer J1.2 (Pin_2)
- net PA13: now also J1.2 (Pin_2), J7.4 (JTMS/SWDIO)
- net PA14: now also J7.6 (JCLK/SWCLK)
- net PA15: now also J7.10 (JTDI/NC)
- net PB3: now also J7.8 (JTDO/SWO)
- net PD8: now also J7.14 (VCP_TX)
- net PD9: now also J7.13 (VCP_RX)
- net ~{RESET}: now also J7.12 (~{RST})
Other:
- company: Kevinbot -> Kevinbot Robotics

Commit message: sch, pcb: FTSH-107-01-L-DV-K-A PN
Parts:
- J7: manf# (none) -> FTSH-107-01-L-DV-K-A
Changed lines of the file:
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@@
+			)
+		)
+		(property "manf#" " FTSH-107-01-L-DV-K-A"
+			(at 440.69 154.94 0)
+			(hide yes)
+			(show_name no)
+			(do_not_autoplace no)
+			(effects
+				(font
+					(size 1.27 1.27)
+				)
 			)
 		)

Commit message: led fixes
Connections:
- net PA7: now also R24.1; no longer R25.1
- net PC8: now also R25.1; no longer R24.1
Changed lines of the file:
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@@
 	)
 	(label "PA7"
-		(at 444.5 78.74 180)
+		(at 455.93 100.33 180)
 		(effects
 			(font
@@
 	)
 	(label "PC8"
-		(at 455.93 100.33 180)
-		(effects
-			(font
+		(at 444.5 78.74 180)
+		(effects
+			(font
